File: 2s/chg-board.kicad_pcb (KiCad board)
At the start: 2 copper layers, 50 x 38 mm, 6 parts, among them J1 Conn_01x09_Male, J2 Conn_01x09_Male, J3 Conn_01x09_Male, J4 Conn_01x09_Male, J5 Conn_01x02_Female, J6 Conn_01x07_Female

Commit message: Some changes to 2s board
Parts:
- J1, J2, J3, J4: footprint custom:xt30_3 -> footprints:xt30_3
